File: board/spark.kicad_pcb (KiCad board)
At the start: 4 copper layers, 198.5 x 85 mm, 43 parts, among them J10 Barrel_Jack, J101 Conn_01x01, J102 Conn_01x01, J103 Conn_01x01, J201 Conn_01x01, J202 Conn_01x01, J203 Conn_01x01, J3 Conn_02x06_Odd_Even, J301 Conn_01x01, J302 Conn_01x01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

Commit message: Release spark-relay-actuator-pi-3.0
Other:
- net class Default removed
- net class Power removed
- net class Thin removed
- board text added: "SPARK-RELAY-ACTUATOR-PI-3.0"
- board text removed: "P/N: SPARK-RELAY-ACTUATOR-PI V2 REV: 1"

Commit message: Release spark-relay-actuator-pi-3.2
Other:
- board text added: "SPARK-RELAY-ACTUATOR-PI-3.2"
- board text removed: "SPARK-RELAY-ACTUATOR-PI-3.0"
Changed lines of the file:
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@@
   (paper "A4")
   (title_block
-    (title "spark-relay-actuator-pi-3.1")
+    (title "spark-relay-actuator-pi-3.2")
     (company "Lightside Instruments AS")
   )
@@
     (effects (font (size 1.5 1.5) (thickness 0.3)))
   )
-  (gr_text "SPARK-RELAY-ACTUATOR-PI-3.0" (at 27.75 96.5) (layer "F.SilkS")
+  (gr_text "SPARK-RELAY-ACTUATOR-PI-3.2" (at 27.75 96.5) (layer "F.SilkS")
     (effects (font (size 1.5 1.5) (thickness 0.3)) (justify left))
   )

Commit message: Release spark4pi-relay-actuator-1.0
Other:
- board text added: "SPARK4PI-RELAY-ACTUATOR-1.0"
- board text removed: "SPARK-RELAY-ACTUATOR-PI-3.2"
Changed lines of the file:
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@@
   (paper "A4")
   (title_block
-    (title "spark-relay-actuator-pi-3.2")
+    (title "spark4pi-relay-actuator-1.0")
     (company "Lightside Instruments AS")
   )
@@
     (effects (font (size 1.5 1.5) (thickness 0.3)))
   )
-  (gr_text "SPARK-RELAY-ACTUATOR-PI-3.2" (at 27.75 96.5) (layer "F.SilkS")
+  (gr_text "SPARK4PI-RELAY-ACTUATOR-1.0" (at 27.75 96.5) (layer "F.SilkS")
     (effects (font (size 1.5 1.5) (thickness 0.3)) (justify left))
   )

Commit message: Release spark4pi-relay-actuator-1.1
Other:
- board text added: "SPARK4PI-RELAY-ACTUATOR-1.1"
- board text removed: "SPARK4PI-RELAY-ACTUATOR-1.0"
Changed lines of the file:
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@@
   (paper "A4")
   (title_block
-    (title "spark4pi-relay-actuator-1.0")
+    (title "spark4pi-relay-actuator-1.1")
     (company "Lightside Instruments AS")
   )
@@
     (effects (font (size 1.5 1.5) (thickness 0.3)))
   )
-  (gr_text "SPARK4PI-RELAY-ACTUATOR-1.0" (at 27.75 96.5) (layer "F.SilkS")
+  (gr_text "SPARK4PI-RELAY-ACTUATOR-1.1" (at 27.75 96.5) (layer "F.SilkS")
     (effects (font (size 1.5 1.5) (thickness 0.3)) (justify left))
   )

Commit message: Release spark4pi-relay-actuator-1.3
Parts:
- removed the REF** at (129.5, 126.0)
- added ?: , spark:Hole_2.5MM, F.Cu at (210.5, 107.5)
- added ?: , spark:Hole_2.5MM, F.Cu at (210.5, 76.0)
Connections:
- net +3V3 renamed +3.3V
- P5 pad 10: (no net) -> unconnected-(P5-Pad10)
- P5 pad 12: (no net) -> unconnected-(P5-Pad12)
- P5 pad 15: (no net) -> PORT4
- P5 pad 18: (no net) -> iCE_CREST
- P5 pad 19: (no net) -> iCE_MOSI
- P5 pad 21: (no net) -> iCE_MISO
- P5 pad 22: (no net) -> iCE_CDONE
- P5 pad 23: (no net) -> iCE_SCK
- P5 pad 24: (no net) -> iCE_SS_B
- P5 pad 26: (no net) -> unconnected-(P5-Pad26)
- P5 pad 27: (no net) -> unconnected-(P5-Pad27)
- P5 pad 28: (no net) -> unconnected-(P5-Pad28)
- P5 pad 29: (no net) -> unconnected-(P5-Pad29)
- P5 pad 3: (no net) -> unconnected-(P5-Pad3)
- P5 pad 31: (no net) -> unconnected-(P5-Pad31)
- P5 pad 32: (no net) -> unconnected-(P5-Pad32)
- P5 pad 33: (no net) -> unconnected-(P5-Pad33)
- P5 pad 35: (no net) -> unconnected-(P5-Pad35)
- P5 pad 36: (no net) -> PORT5
- P5 pad 37: (no net) -> PORT6
- P5 pad 38: (no net) -> REMOTE
- P5 pad 5: (no net) -> unconnected-(P5-Pad5)
- P5 pad 7: (no net) -> unconnected-(P5-Pad7)
- P5 pad 8: (no net) -> unconnected-(P5-Pad8)
Other:
- board text added: "12V-15V -> 5V"
- board text added: "SPARK4PI-RELAY-ACTUATOR-1.3"
- board text removed: "12V -> 5V"
- board text removed: "SPARK4PI-RELAY-ACTUATOR-1.1"

Commit message: Release spark4pi-relay-actuator-1.4
Other:
- board text added: "SPARK4PI-RELAY-ACTUATOR-1.4"
- board text removed: "SPARK4PI-RELAY-ACTUATOR-1.3"

Commit message: Release spark4pi-relay-actuator-2.0
Parts:
- removed the ? at (210.5, 76.0)
- removed the ? at (210.5, 45.0)
- removed the ? at (110.0, 76.0)
- removed the ? at (159.0, 76.0)
- removed the ? at (210.5, 107.5)
- removed REF**: Hole_2.5MM, spark:Hole_2.5MM
- added 1: Fiducial_1mm_Mask3mm, Fiducial:Fiducial_1mm_Mask3mm, F.Cu at (25.0, 44.5)
- added 2: Fiducial_1mm_Mask3mm, Fiducial:Fiducial_1mm_Mask3mm, F.Cu at (205.5, 122.5)
- added ?: , spark:mount_hole, F.Cu at (158.5, 77.5)
- added ?: , spark:mount_hole, F.Cu at (210.5, 102.5)
- added ?: , spark:mount_hole, F.Cu at (210.5, 122.5)
- added ?: , spark:mount_hole, F.Cu at (19.5, 122.5)
- added ?: , spark:mount_hole, F.Cu at (110.5, 77.5)
- added ?: , spark:mount_hole, F.Cu at (210.5, 44.5)
- turned ? to 0 degrees
Other:
- board size 198.5 x 85 mm -> 198 x 85 mm
- board text added: "J103"
- board text added: "J203"
- board text added: "J303"
- board text added: "SPARK4PI-RELAY-ACTUATOR-2.0"
- board text removed: "SPARK4PI-RELAY-ACTUATOR-1.4"
