File: board/spark.kicad_pcb (KiCad board)
At the start: 4 copper layers, 198 x 85 mm, 46 parts, among them J10 Barrel_Jack, J101 Conn_01x01, J102 Conn_01x01, J103 Conn_01x01, J201 Conn_01x01, J202 Conn_01x01, J203 Conn_01x01, J3 Conn_02x06_Odd_Even, J301 Conn_01x01, J302 Conn_01x01, J303 Conn_01x01, J4 Conn_02x06_Odd_Even, K101 G5LE-1, K201 G5LE-1, K301 G5LE-1, P5 Raspberry_Pi_2_3, Q101 BS870, Q201 BS870, Q301 BS870, SW1 SW_Push

Commit message: Release spark4pi-relay-actuator-2.1
Other:
- board text added: "SPARK4PI-RELAY-ACTUATOR-2.1"
- board text removed: "SPARK4PI-RELAY-ACTUATOR-2.0"

Commit message: Release spark4pi-relay-actuator-2.2
Other:
- board text added: "SPARK4PI-RELAY-ACTUATOR-2.2"
- board text removed: "SPARK4PI-RELAY-ACTUATOR-2.1"
Changed lines of the file:
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@@
   (paper "A4")
   (title_block
-    (title "spark4pi-relay-actuator-2.1")
+    (title "spark4pi-relay-actuator-2.2")
     (company "Lightside Instruments AS")
   )
@@
     (effects (font (size 1.5 1.5) (thickness 0.3)))
   )
-  (gr_text "SPARK4PI-RELAY-ACTUATOR-2.1" (at 27.75 96.5) (layer "F.SilkS")
+  (gr_text "SPARK4PI-RELAY-ACTUATOR-2.2" (at 27.75 96.5) (layer "F.SilkS")
     (effects (font (size 1.5 1.5) (thickness 0.3)) (justify left))
   )

Commit message: Release spark4pi-relay-actuator-2.3
Other:
- board text added: "spark4pi-relay-actuator-2.3"
- board text removed: "SPARK4PI-RELAY-ACTUATOR-2.2"
Changed lines of the file:
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@@
   (paper "A4")
   (title_block
-    (title "spark4pi-relay-actuator-2.2")
+    (title "spark4pi-relay-actuator-2.3")
     (company "Lightside Instruments AS")
   )
@@
     (effects (font (size 1.5 1.5) (thickness 0.3)))
   )
-  (gr_text "SPARK4PI-RELAY-ACTUATOR-2.2" (at 27.75 96.5) (layer "F.SilkS")
+  (gr_text "spark4pi-relay-actuator-2.3" (at 27.75 96.5) (layer "F.SilkS")
     (effects (font (size 1.5 1.5) (thickness 0.3)) (justify left))
   )

Commit message: Release spark4pi-digital-io-2.4
Parts:
- removed the ? at (134.5, 68.2)
- removed the ? at (19.5, 122.5)
- removed the ? at (158.5, 77.5)
- removed the ? at (110.5, 77.5)
- removed the ? at (210.5, 44.5)
- removed D201, D301: D_Schottky, Diode_SMD:D_0603_1608Metric
- removed D202, D302: LED, Diode_SMD:D_0603_1608Metric
- removed J10: Barrel_Jack, spark:PJ1-021-SMT-TR
- removed J102, J103, J202, J203, J302, J303: Conn_01x01, spark:banana-plug-horizontal-black
- removed J3, J4: Conn_02x06_Odd_Even, spark:Socket_Strip_SMD_2x6_Pitch2mm
- removed K101, K201, K301: G5LE-1, Relay_THT:Relay_SPDT_Omron-G5LE-1
- removed Q201, Q301: BS870, Package_TO_SOT_SMD:SOT-23
- removed R201, R301: 10K, Resistor_SMD:R_0402_1005Metric
- removed R202, R203, R302, R303: 1K, Resistor_SMD:R_0402_1005Metric
- removed SW1: SW_Push, Button_Switch_THT:SW_Tactile_SPST_Angled_PTS645Vx83-2LFS
- added ?: , , F.Cu at (19.5, 122.5)
- added ?: , spark:lsi-logo-32mm-silks, F.Cu at (39.5, 102.5)
- added ?: , spark:mount_hole, F.Cu at (158.5, 44.5)
- added ?: , spark:mount_hole, F.Cu at (158.5, 102.5)
- added ?: , spark:mount_hole, F.Cu at (110.5, 102.5)
- added ?: , , F.Cu at (210.5, 44.5)
- added ?: , spark:mount_hole, F.Cu at (110.5, 44.5)
- added C1: 10uF, Capacitor_SMD:C_0402_1005Metric, F.Cu at (36.5, 54.0)
- added C101: 10uF, Capacitor_SMD:C_0402_1005Metric, F.Cu at (80.0, 113.0)
- added C102: 10uF, Capacitor_SMD:C_0402_1005Metric, F.Cu at (71.0, 109.5)
- added C2: 10uF, Capacitor_SMD:C_0402_1005Metric, F.Cu at (39.5, 64.5)
- added D1: LED, LED_SMD:LED_0603_1608Metric, F.Cu at (39.5, 124.5)
- added D103: D_TVS, Resistor_SMD:R_0402_1005Metric, F.Cu at (76.5, 115.5)
- added J1: USB_C_Receptacle_USB2.0, Connector_USB:USB_C_Receptacle_GCT_USB4105-xx-A_16P_TopMnt_Horizontal, F.Cu at (39.5, 44.5)
- added J2: Conn_02x03, Connector_PinHeader_2.54mm:PinHeader_2x01_P2.54mm_Vertical, F.Cu at (25.9, 49.4)
- added J401: Conn_01x01_Shielded, spark:SMA_LINX_CONSMA002_Horizontal, F.Cu at (146.5, 121.0)
- added J501: Conn_01x01_Shielded, spark:SMA_LINX_CONSMA002_Horizontal, F.Cu at (170.5, 121.1)
- added J601: Conn_01x01_Shielded, spark:SMA_LINX_CONSMA002_Horizontal, F.Cu at (194.5, 121.0)
- added Q102: Q_NPN_BEC_BRT, Package_TO_SOT_SMD:SOT-323_SC-70, F.Cu at (84.5, 121.0)
- added R1: 1K, Resistor_SMD:R_0402_1005Metric, F.Cu at (37.0, 124.5)
- added R104: 10K, Resistor_SMD:R_0402_1005Metric, F.Cu at (69.0, 112.0)
- added R2: 5.1K, Resistor_SMD:R_0402_1005Metric, F.Cu at (41.5, 51.5)
- added Ref**: Val**, spark:raspberry-pi-signal-interface-silks, F.Cu at (121.2, 49.4)
- added Ref**: Val**, spark:raspberry-pi-signal-interface-silks, F.Cu at (73.2, 49.4)
- added Ref**: Val**, spark:raspberry-pi-signal-interface-silks, F.Cu at (97.2, 49.4)
- added Ref**: Val**, spark:raspberry-pi-signal-interface-silks, F.Cu at (145.2, 49.4)
- added Ref**: Val**, spark:raspberry-pi-signal-interface-silks, F.Cu at (193.2, 49.4)
- added Ref**: Val**, spark:raspberry-pi-signal-interface-silks, F.Cu at (169.2, 49.4)
- added U1: LD1117S33TR_SOT223, Package_TO_SOT_SMD:SOT-223-3_TabPin2, F.Cu at (39.1, 59.0)
- added U101: 74LVC1G125, Package_SO:TSOP-5_1.65x3.05mm_P0.95mm, F.Cu at (77.5, 112.0)
- added U102: 74LVC1G125, Package_SO:TSOP-5_1.65x3.05mm_P0.95mm, F.Cu at (71.5, 112.0)
- added U103: SN74LVC1G14DBV, Package_TO_SOT_SMD:SOT-23-5, F.Cu at (77.5, 108.0)
- 1, 2: value Fiducial_1mm_Mask3mm -> (none); footprint Fiducial:Fiducial_1mm_Mask3mm -> (none)
- D101: value D_Schottky -> LED; footprint Diode_SMD:D_0603_1608Metric -> LED_SMD:LED_0603_1608Metric
- D102: footprint Diode_SMD:D_0603_1608Metric -> LED_SMD:LED_0603_1608Metric
- J101, J201, J301: value Conn_01x01 -> Conn_01x01_Shielded; footprint spark:banana-plug-horizontal-black -> spark:SMA_LINX_CONSMA002_Horizontal
- Q101: value BS870 -> Q_NPN_BEC_BRT; footprint Package_TO_SOT_SMD:SOT-23 -> Package_TO_SOT_SMD:SOT-323_SC-70
- R101: value 10K -> 1K
- R103: value 1K -> 51; footprint Resistor_SMD:R_0402_1005Metric -> Resistor_SMD:R_0805_2012Metric
- moved J301 49.2 mm to (122.5, 121.0), turned to 180 degrees
- moved D101 40.8 mm to (67.5, 124.5)
- moved R102 40.7 mm to (84.0, 124.5), turned to 180 degrees
- moved R101 37.4 mm to (65.0, 124.5)
- moved Q101 36.2 mm to (64.5, 121.0), turned to -90 degrees
- moved J201 27.3 mm to (97.5, 121.0), turned to 180 degrees
- moved R103 15.5 mm to (74.5, 114.5)
- moved J101 11.0 mm to (74.5, 121.0), turned to 180 degrees
- moved 2 6.81 mm to (210.5, 117.9)
- moved D102 5.02 mm to (81.5, 124.5), turned to 0 degrees
- moved 1 0.79 mm to (24.2, 44.5)
Connections:
- D101 pad 1: SYS_DCIN -> Net-(D101-Pad1)
- D102 pad 2: SYS_DCIN -> Net-(D102-Pad2)
- J101 pad 1: Net-(J101-Pad1) -> Net-(D103-Pad1)
- J201 pad 1: Net-(J201-Pad1) -> unconnected-(J201-Pad1)
- J301 pad 1: Net-(J301-Pad1) -> unconnected-(J301-Pad1)
- P5 pad 12: unconnected-(P5-Pad12) -> PORT1_TX_ENABLE
- Q101 pad 1: Net-(Q101-Pad1) -> PORT1
- Q101 pad 3: Net-(D101-Pad2) -> Net-(D101-Pad1)
- R101 pad 1: Net-(Q101-Pad1) -> +3V3
- R101 pad 2: GND -> Net-(D101-Pad2)
- R102 pad 1: PORT1 -> +3V3
- R102 pad 2: Net-(Q101-Pad1) -> Net-(D102-Pad2)
- R103 pad 1: Net-(D102-Pad1) -> Net-(D103-Pad1)
- R103 pad 2: Net-(D101-Pad2) -> Net-(R103-Pad2)
Routing:
- net SYS_DCIN: track 345.4 -> 0.00 mm, vias 14 -> 0
- net GND: track 195.5 -> 17.6 mm, vias 20 -> 3
- net PORT3: track 158.2 -> 0.00 mm
- net PORT1_TX_ENABLE: track 0.00 -> 131.3 mm, vias 0 -> 3
- net PORT2: track 113.7 -> 0.00 mm
- net Net-(D301-Pad2): track 69.0 -> 0.00 mm, vias 1 -> 0
- net Net-(D201-Pad2): track 69.0 -> 0.00 mm, vias 1 -> 0
- net Net-(D101-Pad2): track 69.0 -> 1.19 mm, vias 1 -> 0
- net PORT1: track 70.0 -> 125.8 mm, vias 0 -> 1
- net +5V: track 0.00 -> 33.7 mm, vias 6 -> 2
- net RESET_BTN: track 32.2 -> 0.00 mm
- net +3.3V: track 0.00 -> 30.1 mm
- net IN3: track 25.0 -> 0.00 mm
- net IN2: track 25.0 -> 0.00 mm
- net IN1: track 25.0 -> 0.00 mm
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- added copper zone on In2.Cu, net +3V3
- added copper zone on B.Cu, net GND
- removed copper zone on B.Cu, net +5V
- removed copper zone on F.Cu, net +5V
- removed copper zone on B.Cu, net IN1
- removed copper zone on B.Cu, net IN2
- removed copper zone on B.Cu, net IN3
- removed copper zone on B.Cu, net Net-(J101-Pad1)
- removed copper zone on B.Cu, net Net-(J102-Pad1)
- removed copper zone on B.Cu, net Net-(J201-Pad1)
- removed copper zone on B.Cu, net Net-(J202-Pad1)
- removed copper zone on B.Cu, net Net-(J301-Pad1)
- removed copper zone on B.Cu, net Net-(J302-Pad1)
- removed copper zone on F.Cu, net SYS_DCIN
- removed copper zone on In2.Cu, net SYS_DCIN
Other:
- board text added: "!!!"
- board text added: "power"
- board text added: "spark4pi-digital-io-1.0"
- board text removed: "1"
- board text removed: "12V-15V -> 5V"
- board text removed: "2"
- board text removed: "27x16 mm"
- board text removed: "3"
- board text removed: "A"
- board text removed: "B"
- board text removed: "J103"
- board text removed: "J203"
- board text removed: "J303"
- board text removed: "spark4pi-relay-actuator-2.3"

Commit message: Release spark4pi-digital-io-2.5
Parts:
- added C201: 100nF, Capacitor_SMD:C_0402_1005Metric, F.Cu at (104.0, 113.0)
- added C202: 100nF, Capacitor_SMD:C_0402_1005Metric, F.Cu at (95.0, 109.5)
- added C301: 100nF, Capacitor_SMD:C_0402_1005Metric, F.Cu at (128.0, 113.0)
- added C302: 100nF, Capacitor_SMD:C_0402_1005Metric, F.Cu at (119.0, 109.5)
- added C401: 100nF, Capacitor_SMD:C_0402_1005Metric, F.Cu at (152.0, 113.0)
- added C402: 100nF, Capacitor_SMD:C_0402_1005Metric, F.Cu at (143.0, 109.5)
- added C501: 100nF, Capacitor_SMD:C_0402_1005Metric, F.Cu at (176.0, 113.0)
- added C502: 100nF, Capacitor_SMD:C_0402_1005Metric, F.Cu at (167.0, 109.5)
- added C601: 100nF, Capacitor_SMD:C_0402_1005Metric, F.Cu at (200.0, 113.0)
- added C602: 100nF, Capacitor_SMD:C_0402_1005Metric, F.Cu at (191.0, 109.5)
- added D201: LED, LED_SMD:LED_0603_1608Metric, F.Cu at (91.5, 124.5)
- added D202: LED, LED_SMD:LED_0603_1608Metric, F.Cu at (105.5, 124.5)
- added D203: D_TVS, Resistor_SMD:R_0402_1005Metric, F.Cu at (100.5, 115.5)
- added D301: LED, LED_SMD:LED_0603_1608Metric, F.Cu at (115.5, 124.5)
- added D302: LED, LED_SMD:LED_0603_1608Metric, F.Cu at (129.5, 124.5)
- added D303: D_TVS, Resistor_SMD:R_0402_1005Metric, F.Cu at (124.5, 115.5)
- added D401: LED, LED_SMD:LED_0603_1608Metric, F.Cu at (139.5, 124.5)
- added D402: LED, LED_SMD:LED_0603_1608Metric, F.Cu at (153.5, 124.5)
- added D403: D_TVS, Resistor_SMD:R_0402_1005Metric, F.Cu at (148.5, 115.5)
- added D501: LED, LED_SMD:LED_0603_1608Metric, F.Cu at (163.5, 124.5)
- added D502: LED, LED_SMD:LED_0603_1608Metric, F.Cu at (177.5, 124.5)
- added D503: D_TVS, Resistor_SMD:R_0402_1005Metric, F.Cu at (172.5, 115.5)
- added D601: LED, LED_SMD:LED_0603_1608Metric, F.Cu at (187.5, 124.5)
- added D602: LED, LED_SMD:LED_0603_1608Metric, F.Cu at (201.5, 124.5)
- added D603: D_TVS, Resistor_SMD:R_0402_1005Metric, F.Cu at (196.5, 115.5)
- added Q201: Q_NPN_BEC_BRT, Package_TO_SOT_SMD:SOT-323_SC-70, F.Cu at (88.5, 121.0)
- added Q202: Q_NPN_BEC_BRT, Package_TO_SOT_SMD:SOT-323_SC-70, F.Cu at (108.5, 121.0)
- added Q301: Q_NPN_BEC_BRT, Package_TO_SOT_SMD:SOT-323_SC-70, F.Cu at (112.5, 121.0)
- added Q302: Q_NPN_BEC_BRT, Package_TO_SOT_SMD:SOT-323_SC-70, F.Cu at (132.5, 121.0)
- added Q401: Q_NPN_BEC_BRT, Package_TO_SOT_SMD:SOT-323_SC-70, F.Cu at (136.5, 121.0)
- added Q402: Q_NPN_BEC_BRT, Package_TO_SOT_SMD:SOT-323_SC-70, F.Cu at (156.5, 121.0)
- added Q501: Q_NPN_BEC_BRT, Package_TO_SOT_SMD:SOT-323_SC-70, F.Cu at (160.5, 121.0)
- added Q502: Q_NPN_BEC_BRT, Package_TO_SOT_SMD:SOT-323_SC-70, F.Cu at (180.5, 121.0)
- added Q601: Q_NPN_BEC_BRT, Package_TO_SOT_SMD:SOT-323_SC-70, F.Cu at (184.5, 121.0)
- added Q602: Q_NPN_BEC_BRT, Package_TO_SOT_SMD:SOT-323_SC-70, F.Cu at (204.5, 121.0)
- added R201: 1K, Resistor_SMD:R_0402_1005Metric, F.Cu at (89.0, 124.5)
- added R202: 1K, Resistor_SMD:R_0402_1005Metric, F.Cu at (108.0, 124.5)
- added R203: 51, Resistor_SMD:R_0805_2012Metric, F.Cu at (98.5, 114.5)
- added R204: 10K, Resistor_SMD:R_0402_1005Metric, F.Cu at (93.0, 112.0)
- added R301: 1K, Resistor_SMD:R_0402_1005Metric, F.Cu at (113.0, 124.5)
- added R302: 1K, Resistor_SMD:R_0402_1005Metric, F.Cu at (132.0, 124.5)
- added R303: 51, Resistor_SMD:R_0805_2012Metric, F.Cu at (122.5, 114.5)
- added R304: 10K, Resistor_SMD:R_0402_1005Metric, F.Cu at (117.0, 112.0)
- added R401: 1K, Resistor_SMD:R_0402_1005Metric, F.Cu at (137.0, 124.5)
- added R402: 1K, Resistor_SMD:R_0402_1005Metric, F.Cu at (156.0, 124.5)
- added R403: 51, Resistor_SMD:R_0805_2012Metric, F.Cu at (146.5, 114.5)
- added R404: 10K, Resistor_SMD:R_0402_1005Metric, F.Cu at (141.0, 112.0)
- added R501: 1K, Resistor_SMD:R_0402_1005Metric, F.Cu at (161.0, 124.5)
- added R502: 1K, Resistor_SMD:R_0402_1005Metric, F.Cu at (180.0, 124.5)
- added R503: 51, Resistor_SMD:R_0805_2012Metric, F.Cu at (170.5, 114.5)
- added R504: 10K, Resistor_SMD:R_0402_1005Metric, F.Cu at (165.0, 112.0)
- added R601: 1K, Resistor_SMD:R_0402_1005Metric, F.Cu at (185.0, 124.5)
- added R602: 1K, Resistor_SMD:R_0402_1005Metric, F.Cu at (204.0, 124.5)
- added R603: 51, Resistor_SMD:R_0805_2012Metric, F.Cu at (194.5, 114.5)
- added R604: 10K, Resistor_SMD:R_0402_1005Metric, F.Cu at (189.0, 112.0)
- added U201: 74LVC1G125, Package_SO:TSOP-5_1.65x3.05mm_P0.95mm, F.Cu at (101.5, 112.0)
- added U202: 74LVC1G125, Package_SO:TSOP-5_1.65x3.05mm_P0.95mm, F.Cu at (95.5, 112.0)
- added U203: SN74LVC1G14DBV, Package_TO_SOT_SMD:SOT-23-5, F.Cu at (101.5, 108.0)
- added U301: 74LVC1G125, Package_SO:TSOP-5_1.65x3.05mm_P0.95mm, F.Cu at (125.5, 112.0)
- added U302: 74LVC1G125, Package_SO:TSOP-5_1.65x3.05mm_P0.95mm, F.Cu at (119.5, 112.0)
- added U303: SN74LVC1G14DBV, Package_TO_SOT_SMD:SOT-23-5, F.Cu at (125.5, 108.0)
- added U401: 74LVC1G125, Package_SO:TSOP-5_1.65x3.05mm_P0.95mm, F.Cu at (149.5, 112.0)
- added U402: 74LVC1G125, Package_SO:TSOP-5_1.65x3.05mm_P0.95mm, F.Cu at (143.5, 112.0)
- added U403: SN74LVC1G14DBV, Package_TO_SOT_SMD:SOT-23-5, F.Cu at (149.5, 108.0)
- added U501: 74LVC1G125, Package_SO:TSOP-5_1.65x3.05mm_P0.95mm, F.Cu at (173.5, 112.0)
- added U502: 74LVC1G125, Package_SO:TSOP-5_1.65x3.05mm_P0.95mm, F.Cu at (167.5, 112.0)
- added U503: SN74LVC1G14DBV, Package_TO_SOT_SMD:SOT-23-5, F.Cu at (173.5, 108.0)
- added U601: 74LVC1G125, Package_SO:TSOP-5_1.65x3.05mm_P0.95mm, F.Cu at (197.5, 112.0)
- added U602: 74LVC1G125, Package_SO:TSOP-5_1.65x3.05mm_P0.95mm, F.Cu at (191.5, 112.0)
- added U603: SN74LVC1G14DBV, Package_TO_SOT_SMD:SOT-23-5, F.Cu at (197.5, 108.0)
- C101, C102: value 10uF -> 100nF
- moved C2 10.5 mm to (40.5, 54.0)
- moved J201 1.00 mm to (98.5, 121.0)
- moved U1 0.15 mm to (39.0, 59.0)
- moved J501 0.08 mm to (170.5, 121.0)
Connections:
- J201 pad 1: unconnected-(J201-Pad1) -> Net-(J201-Pad1)
- J301 pad 1: unconnected-(J301-Pad1) -> Net-(J301-Pad1)
- J401 pad 1: unconnected-(J401-Pad1) -> Net-(J401-Pad1)
- J501 pad 1: unconnected-(J501-Pad1) -> Net-(J501-Pad1)
- J601 pad 1: unconnected-(J601-Pad1) -> Net-(J601-Pad1)
- P5 pad 29: unconnected-(P5-Pad29) -> PORT2_TX_ENABLE
- P5 pad 31: unconnected-(P5-Pad31) -> PORT3_TX_ENABLE
- P5 pad 32: unconnected-(P5-Pad32) -> PORT4_TX_ENABLE
- P5 pad 33: unconnected-(P5-Pad33) -> PORT5_TX_ENABLE
- P5 pad 35: unconnected-(P5-Pad35) -> PORT6_TX_ENABLE
Routing:
- net PORT6_TX_ENABLE: track 0.00 -> 221.6 mm, vias 0 -> 3
- net PORT6: track 0.00 -> 212.5 mm, vias 0 -> 1
- net PORT5_TX_ENABLE: track 0.00 -> 200.1 mm, vias 0 -> 3
- net PORT4: track 0.00 -> 193.5 mm, vias 0 -> 1
- net PORT5: track 0.00 -> 188.0 mm, vias 0 -> 1
- net PORT4_TX_ENABLE: track 0.00 -> 175.6 mm, vias 0 -> 3
- net PORT3: track 0.00 -> 170.0 mm, vias 0 -> 1
- net PORT3_TX_ENABLE: track 0.00 -> 154.7 mm, vias 0 -> 3
- net PORT2: track 0.00 -> 148.0 mm, vias 0 -> 1
- net PORT2_TX_ENABLE: track 0.00 -> 133.2 mm, vias 0 -> 3
- net +3V3: track 18.0 -> 73.4 mm, vias 9 -> 36
- net GND: track 17.6 -> 71.4 mm, vias 3 -> 20
- net Net-(J601-Pad1): track 0.00 -> 7.11 mm
- net Net-(J501-Pad1): track 0.00 -> 7.11 mm
- net Net-(J401-Pad1): track 0.00 -> 7.11 mm
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Other:
- board text added: "spark4pi-digital-io-2.5"
- board text removed: "spark4pi-digital-io-1.0"

Commit message: Release spark4pi-digital-io-2.6
Routing:
- net GND: vias 20 -> 59
Other:
- board text added: "spark4pi-digital-io-2.6"
- board text removed: "spark4pi-digital-io-2.5"

Commit message: Release spark4pi-digital-io-2.7
Routing:
- net PORT1: track 125.5 -> 214.0 mm
- net PORT2: track 148.0 -> 214.0 mm
- net PORT3: track 170.0 -> 214.9 mm
- net PORT5: track 188.0 -> 214.9 mm
- net PORT4: track 193.5 -> 214.0 mm
- net PORT6: track 212.5 -> 214.1 mm
Other:
- board text added: "spark4pi-digital-io-2.7"
- board text removed: "spark4pi-digital-io-2.6"

Commit message: Release spark4pi-digital-io-2.8
Parts:
- added J3: Conn_01x03, Connector_PinHeader_2.54mm:PinHeader_1x03_P2.54mm_Vertical, F.Cu at (51.2, 49.4)
- D1: value LED -> LED_WHITE
- D101, D201, D301, D401, D501, D601: value LED -> LED_GREEN
- D102, D202, D302, D402, D502, D602: value LED -> LED_BLUE
- J2: value Conn_02x03 -> Conn_01x02
Connections:
- C101 pad 1: +3V3 -> Vdrive
- C201 pad 1: +3V3 -> Vdrive
- C301 pad 1: +3V3 -> Vdrive
- C401 pad 1: +3V3 -> Vdrive
- C501 pad 1: +3V3 -> Vdrive
- C601 pad 1: +3V3 -> Vdrive
- U101 pad 5: +3V3 -> Vdrive
- U201 pad 5: +3V3 -> Vdrive
- U301 pad 5: +3V3 -> Vdrive
- U401 pad 5: +3V3 -> Vdrive
- U501 pad 5: +3V3 -> Vdrive
- U601 pad 5: +3V3 -> Vdrive
Routing:
- net Vdrive: track 0.00 -> 284.7 mm, vias 0 -> 10
- net +3V3: track 73.4 -> 57.2 mm, vias 36 -> 30
- net +5V: track 33.7 -> 43.2 mm
Other:
- board text added: "Open (default). Closed - !!! U1 3V3 drives pins 1 and 17."
- board text added: "Select output driver voltage 5V | 3.3V"
- board text added: "spark4pi-digital-io-2.8"
- board text removed: "spark4pi-digital-io-2.7"
