File: board/spark.kicad_pcb (KiCad board)
At the start: 4 copper layers, 198 x 85 mm, 119 parts, among them J1 USB_C_Receptacle_USB2.0, J101 Conn_01x01_Shielded, J2 Conn_01x02, J201 Conn_01x01_Shielded, J3 Conn_01x03, J301 Conn_01x01_Shielded, J401 Conn_01x01_Shielded, J501 Conn_01x01_Shielded, J601 Conn_01x01_Shielded, P5 Raspberry_Pi_2_3, Q101 Q_NPN_BEC_BRT, Q102 Q_NPN_BEC_BRT, Q201 Q_NPN_BEC_BRT, Q202 Q_NPN_BEC_BRT, Q301 Q_NPN_BEC_BRT, Q302 Q_NPN_BEC_BRT, Q401 Q_NPN_BEC_BRT, Q402 Q_NPN_BEC_BRT, Q501 Q_NPN_BEC_BRT, Q502 Q_NPN_BEC_BRT, Q601 Q_NPN_BEC_BRT, Q602 Q_NPN_BEC_BRT, U1 LD1117S33TR_SOT223, U101 74LVC1G125, U102 74LVC1G125, U103 SN74LVC1G14DBV, U201 74LVC1G125, U202 74LVC1G125, U203 SN74LVC1G14DBV, U301 74LVC1G125, U302 74LVC1G125, U303 SN74LVC1G14DBV, U401 74LVC1G125, U402 74LVC1G125, U403 SN74LVC1G14DBV, U501 74LVC1G125, U502 74LVC1G125, U503 SN74LVC1G14DBV, U601 74LVC1G125, U602 74LVC1G125, U603 SN74LVC1G14DBV

Commit message: Release spark4pi-digital-io-2.9
Routing:
- net PORT5_TX_ENABLE: track 200.1 -> 201.6 mm
Other:
- board text added: "spark4pi-digital-io-2.9"
- board text removed: "spark4pi-digital-io-2.8"

Commit message: Release spark4pi-digital-io-2.10
Parts:
- added C104: 100nF, Capacitor_SMD:C_0402_1005Metric, F.Cu at (69.5, 113.0)
- added C204: 100nF, Capacitor_SMD:C_0402_1005Metric, F.Cu at (93.5, 113.0)
- added C3: 10uF, Capacitor_SMD:C_0402_1005Metric, F.Cu at (36.5, 69.0)
- added C304: 100nF, Capacitor_SMD:C_0402_1005Metric, F.Cu at (117.5, 113.0)
- added C4: 10uF, Capacitor_SMD:C_0402_1005Metric, F.Cu at (40.5, 69.0)
- added C404: 100nF, Capacitor_SMD:C_0402_1005Metric, F.Cu at (141.5, 113.0)
- added C504: 100nF, Capacitor_SMD:C_0402_1005Metric, F.Cu at (165.5, 113.0)
- added C604: 100nF, Capacitor_SMD:C_0402_1005Metric, F.Cu at (189.5, 113.0)
- added J4: Conn_01x03, Connector_PinHeader_2.54mm:PinHeader_1x03_P2.54mm_Vertical, F.Cu at (51.3, 56.6)
- added R3: 220, Resistor_SMD:R_0402_1005Metric, F.Cu at (43.5, 72.5)
- added R4: 68, Resistor_SMD:R_0402_1005Metric, F.Cu at (43.5, 70.5)
- added R5: 5.1K, Resistor_SMD:R_0402_1005Metric, F.Cu at (42.5, 52.6)
- added U2: LM317_SOT-223, Package_TO_SOT_SMD:SOT-223-3_TabPin2, F.Cu at (39.0, 74.0)
- U102, U202, U302, U402, U502, U602: value 74LVC1G125 -> TXU0101DCK; footprint Package_SO:TSOP-5_1.65x3.05mm_P0.95mm -> Package_TO_SOT_SMD:SOT-363_SC-70-6
- moved R104 11.4 mm to (80.0, 109.0), turned to 90 degrees
- moved R204 11.4 mm to (104.0, 109.0), turned to 90 degrees
- moved R304 11.4 mm to (128.0, 109.0), turned to 90 degrees
- moved R404 11.4 mm to (152.0, 109.0), turned to 90 degrees
- moved R504 11.4 mm to (176.0, 109.0), turned to 90 degrees
- moved R604 11.4 mm to (200.0, 109.0), turned to 90 degrees
- moved C102 2.12 mm to (69.5, 111.0), turned to -90 degrees
- moved C202 2.12 mm to (93.5, 111.0), turned to -90 degrees
- moved C302 2.12 mm to (117.5, 111.0), turned to -90 degrees
- moved C402 2.12 mm to (141.5, 111.0), turned to -90 degrees
- moved C502 2.12 mm to (165.5, 111.0), turned to -90 degrees
- moved C602 2.12 mm to (189.5, 111.0), turned to -90 degrees
- moved R2 1.00 mm to (42.5, 51.6)
- turned ? to 0 degrees (x2)
Connections:
- J1 pad B5: Net-(J1-PadA5) -> Net-(J1-PadB5)
- U102 pad 1: PORT1_TX_ENABLE -> Vrx
- U102 pad 2: Net-(R103-Pad2) -> GND
- U102 pad 3: GND -> Net-(R103-Pad2)
- U102 pad 5: +3V3 -> Net-(U101-Pad1)
- U202 pad 1: PORT2_TX_ENABLE -> Vrx
- U202 pad 2: Net-(R203-Pad2) -> GND
- U202 pad 3: GND -> Net-(R203-Pad2)
- U202 pad 5: +3V3 -> Net-(U201-Pad1)
- U302 pad 1: PORT3_TX_ENABLE -> Vrx
- U302 pad 2: Net-(R303-Pad2) -> GND
- U302 pad 3: GND -> Net-(R303-Pad2)
- U302 pad 5: +3V3 -> Net-(U301-Pad1)
- U402 pad 1: PORT4_TX_ENABLE -> Vrx
- U402 pad 2: Net-(R403-Pad2) -> GND
- U402 pad 3: GND -> Net-(R403-Pad2)
- U402 pad 5: +3V3 -> Net-(U401-Pad1)
- U502 pad 1: PORT5_TX_ENABLE -> Vrx
- U502 pad 2: Net-(R503-Pad2) -> GND
- U502 pad 3: GND -> Net-(R503-Pad2)
- U502 pad 5: +3V3 -> Net-(U501-Pad1)
- U602 pad 1: PORT6_TX_ENABLE -> Vrx
- U602 pad 2: Net-(R603-Pad2) -> GND
- U602 pad 3: GND -> Net-(R603-Pad2)
- U602 pad 5: +3V3 -> Net-(U601-Pad1)
Routing:
- net Vrx: track 0.00 -> 290.4 mm, vias 0 -> 10
- net +1V65: track 0.00 -> 31.0 mm
- net GND: track 71.4 -> 48.5 mm, vias 59 -> 65
- net +5V: track 43.2 -> 60.5 mm
- net PORT5_TX_ENABLE: track 201.6 -> 190.2 mm, vias 3 -> 1
- net PORT6_TX_ENABLE: track 221.6 -> 210.2 mm, vias 3 -> 1
- net PORT3_TX_ENABLE: track 154.7 -> 143.3 mm, vias 3 -> 1
- net PORT2_TX_ENABLE: track 133.2 -> 121.9 mm, vias 3 -> 1
- net PORT1_TX_ENABLE: track 130.5 -> 119.1 mm, vias 3 -> 1
- net PORT4_TX_ENABLE: track 175.6 -> 164.6 mm, vias 3 -> 1
- net Net-(U301-Pad1): track 2.61 -> 10.6 mm
- net Net-(U201-Pad1): track 2.61 -> 10.6 mm
- net Net-(U101-Pad1): track 2.61 -> 10.6 mm
- net Net-(U501-Pad1): track 2.61 -> 10.6 mm
- net Net-(U401-Pad1): track 2.61 -> 10.6 mm
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Other:
- board text added: "O"
- board text added: "Q_NPN_BEC_BRT"
- board text added: "Select receiver voltage 1.65V | 3.3V"
- board text added: "X"
- board text added: "spark4pi-digital-io-2.10"
- board text removed: "spark4pi-digital-io-2.9"
