File: board/spark.kicad_sch (KiCad schematic)
At the start: 35 parts, among them J10 Barrel_Jack, J101 Conn_01x01, J102 Conn_01x01, J103 Conn_01x01, J201 Conn_01x01, J202 Conn_01x01, J203 Conn_01x01, J3 Conn_02x06_Odd_Even, J301 Conn_01x01, J302 Conn_01x01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

Commit message: Release spark-relay-actuator-pi-3.1
Other:
- title: spark-relay-actuator-pi-3.0 -> spark-relay-actuator-pi-3.1
Changed lines of the file:
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@@
   (paper "A2")
   (title_block
-    (title "spark-relay-actuator-pi-3.0")
+    (title "spark-relay-actuator-pi-3.1")
     (company "Lightside Instruments AS")
   )

Commit message: Release spark-relay-actuator-pi-3.2
Other:
- title: spark-relay-actuator-pi-3.1 -> spark-relay-actuator-pi-3.2
Changed lines of the file:
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@@
   (paper "A2")
   (title_block
-    (title "spark-relay-actuator-pi-3.1")
+    (title "spark-relay-actuator-pi-3.2")
     (company "Lightside Instruments AS")
   )

Commit message: Release spark4pi-relay-actuator-1.0
Other:
- title: spark-relay-actuator-pi-3.2 -> spark4pi-relay-actuator-1.0
Changed lines of the file:
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@@
   (paper "A2")
   (title_block
-    (title "spark-relay-actuator-pi-3.2")
+    (title "spark4pi-relay-actuator-1.0")
     (company "Lightside Instruments AS")
   )

Commit message: Release spark4pi-relay-actuator-1.1
Other:
- title: spark4pi-relay-actuator-1.0 -> spark4pi-relay-actuator-1.1
Changed lines of the file:
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@@
   (paper "A2")
   (title_block
-    (title "spark4pi-relay-actuator-1.0")
+    (title "spark4pi-relay-actuator-1.1")
     (company "Lightside Instruments AS")
   )

Commit message: Release spark4pi-relay-actuator-1.3
Other:
- title: spark4pi-relay-actuator-1.1 -> spark4pi-relay-actuator-1.3
Changed lines of the file:
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@@
   (paper "A2")
   (title_block
-    (title "spark4pi-relay-actuator-1.1")
+    (title "spark4pi-relay-actuator-1.3")
     (company "Lightside Instruments AS")
   )

Commit message: Release spark4pi-relay-actuator-1.4
Other:
- title: spark4pi-relay-actuator-1.3 -> spark4pi-relay-actuator-1.4
Changed lines of the file:
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@@
   (paper "A2")
   (title_block
-    (title "spark4pi-relay-actuator-1.3")
+    (title "spark4pi-relay-actuator-1.4")
     (company "Lightside Instruments AS")
   )

Commit message: Release spark4pi-relay-actuator-2.0
Other:
- title: spark4pi-relay-actuator-1.4 -> spark4pi-relay-actuator-2.0
Changed lines of the file:
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@@
   (paper "A2")
   (title_block
-    (title "spark4pi-relay-actuator-1.4")
+    (title "spark4pi-relay-actuator-2.0")
     (company "Lightside Instruments AS")
   )

Commit message: Release spark4pi-relay-actuator-2.1
Other:
- title: spark4pi-relay-actuator-2.0 -> spark4pi-relay-actuator-2.1
Changed lines of the file:
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@@
   (paper "A2")
   (title_block
-    (title "spark4pi-relay-actuator-2.0")
+    (title "spark4pi-relay-actuator-2.1")
     (company "Lightside Instruments AS")
   )
