File: board/spark.kicad_sch (KiCad schematic)
At the start: 35 parts, among them J10 Barrel_Jack, J101 Conn_01x01, J102 Conn_01x01, J103 Conn_01x01, J201 Conn_01x01, J202 Conn_01x01, J203 Conn_01x01, J3 Conn_02x06_Odd_Even, J301 Conn_01x01, J302 Conn_01x01, J303 Conn_01x01, J4 Conn_02x06_Odd_Even, K101 G5LE-1, K201 G5LE-1, K301 G5LE-1, P5 Raspberry_Pi_2_3, Q101 BS870, Q201 BS870, Q301 BS870, SW1 SW_Push

Commit message: Release spark4pi-relay-actuator-2.2
Other:
- title: spark4pi-relay-actuator-2.1 -> spark4pi-relay-actuator-2.2
Changed lines of the file:
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@@
   (paper "A2")
   (title_block
-    (title "spark4pi-relay-actuator-2.1")
+    (title "spark4pi-relay-actuator-2.2")
     (company "Lightside Instruments AS")
   )

Commit message: Release spark4pi-relay-actuator-2.3
Other:
- title: spark4pi-relay-actuator-2.2 -> spark4pi-relay-actuator-2.3
Changed lines of the file:
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@@
   (paper "A2")
   (title_block
-    (title "spark4pi-relay-actuator-2.2")
+    (title "spark4pi-relay-actuator-2.3")
     (company "Lightside Instruments AS")
   )

Commit message: Release spark4pi-digital-io-2.4
Parts:
- removed D101, D201, D301: D_Schottky, Diode_SMD:D_0603_1608Metric, symbol Device:D_Schottky
- removed D202, D302: LED, Diode_SMD:D_0603_1608Metric, symbol Device:LED
- removed J10: Barrel_Jack, spark:PJ1-021-SMT-TR, symbol Connector:Barrel_Jack_Switch
- removed J101, J102, J103, J201, J202, J203, J301, J302, J303: Conn_01x01, spark:banana-plug-horizontal-black, symbol Connector_Generic:Conn_01x01
- removed J3, J4: Conn_02x06_Odd_Even, spark:Socket_Strip_SMD_2x6_Pitch2mm, symbol Connector_Generic:Conn_02x06_Odd_Even
- removed K101, K201, K301: G5LE-1, Relay_THT:Relay_SPDT_Omron-G5LE-1, symbol Relay:G5LE-1
- removed Q101, Q201, Q301: BS870, Package_TO_SOT_SMD:SOT-23, symbol spark:BS870-Transistor_FET
- removed R201, R301: 10K, Resistor_SMD:R_0402_1005Metric, symbol Device:R
- removed R202, R203, R302, R303: 1K, Resistor_SMD:R_0402_1005Metric, symbol Device:R
- removed SW1: SW_Push, Button_Switch_THT:SW_Tactile_SPST_Angled_PTS645Vx83-2LFS, symbol Switch:SW_Push
- added C1, C101, C102, C2: 10uF, Capacitor_SMD:C_0402_1005Metric, symbol Device:C_Small
- added D1, D101: LED, LED_SMD:LED_0603_1608Metric, symbol Device:LED
- added D103: D_TVS, Resistor_SMD:R_0402_1005Metric, symbol Device:D_TVS
- added J1: USB_C_Receptacle_USB2.0, Connector_USB:USB_C_Receptacle_GCT_USB4105-xx-A_16P_TopMnt_Horizontal, symbol Connector:USB_C_Receptacle_USB2.0
- added J101, J201, J301, J401, J501, J601: Conn_01x01_Shielded, spark:SMA_LINX_CONSMA002_Horizontal, symbol Connector_Generic_Shielded:Conn_01x01_Shielded
- added J2: Conn_02x03, Connector_PinHeader_2.54mm:PinHeader_2x01_P2.54mm_Vertical, symbol Connector_Generic:Conn_01x02
- added Q101, Q102: Q_NPN_BEC_BRT, Package_TO_SOT_SMD:SOT-323_SC-70, symbol Device:Q_NPN_BEC_BRT
- added R1: 1K, Resistor_SMD:R_0402_1005Metric, symbol Device:R
- added R104: 10K, Resistor_SMD:R_0402_1005Metric, symbol Device:R
- added R2: 5.1K, Resistor_SMD:R_0402_1005Metric, symbol Device:R
- added U1: LD1117S33TR_SOT223, Package_TO_SOT_SMD:SOT-223-3_TabPin2, symbol Regulator_Linear:LD1117S33TR_SOT223
- added U101, U102: 74LVC1G125, Package_SO:TSOP-5_1.65x3.05mm_P0.95mm, symbol ice4pi:74LVC1G125
- added U103: SN74LVC1G14DBV, Package_TO_SOT_SMD:SOT-23-5, symbol 74xGxx:SN74LVC1G14DBV
- D102: footprint Diode_SMD:D_0603_1608Metric -> LED_SMD:LED_0603_1608Metric
- R101: value 10K -> 1K
- R103: value 1K -> 51; footprint Resistor_SMD:R_0402_1005Metric -> Resistor_SMD:R_0805_2012Metric
Connections:
- net +12V is gone; now on an unnamed net: D102.2 (A)
- net +3.3V: now also J2.1 (Pin_1)
- net +5V: now also C1.1, J1.A4 (VBUS), J1.A9 (VBUS), J1.B4 (VBUS), J1.B9 (VBUS), U1.3 (VI)
- net GND: now also C1.2, C101.2, C102.2, C2.2, D1.1 (K), D103.2 (A2), J1.A1 (GND), J1.A12 (GND), J1.B1 (GND), J1.B12 (GND), J1.S1 (SHIELD), J101.SH (Shield), J201.SH (Shield), J301.SH (Shield), J401.SH (Shield), J501.SH (Shield), J601.SH (Shield), Q101.2 (E), Q102.2 (E), R2.2, U1.1 (GND), U101.3 (GND), U102.3 (GND), U103.3 (GND); no longer R101.2
- net PORT1: now also Q101.1 (B), U101.2 (D), U102.4 (O); no longer R102.1
- net at R103.2: now also U101.4 (O), U102.2 (D)
- net at R102.2: no longer R101.1
- net at R103.1: now also D103.1 (A1), J101.1 (Pin_1); no longer D102.1 (K)
- net PORT1_TX_ENABLE: now reaches P5.12 (GPIO18/PWM0)
- net PORT1_TX_ENABLE: now also Q102.1 (B), R104.2, U102.1 (EN), U103.2
- new net: U101.1 (EN), U103.4
- new net: J1.A5 (CC1), J1.B5 (CC2), R2.1
- new net: D101.1 (K), Q101.3 (C)
- new net: D101.2 (A), R101.2
- new net: D102.1 (K), Q102.3 (C)
- new net: D1.2 (A), R1.2
- new net +3V3: C101.1, C102.1, C2.1, J2.2 (Pin_2), R1.1, R101.1, R102.1, R104.1, U1.2 (VO), U101.5 (VCC), U102.5 (VCC), U103.5 (VCC)
Other:
- note added: "Jumper: Default open. Power the 2x20 Raspberry Pi 3.3V rail from the LDO regulator on the extension board - 3V3 800 mA. Leave open if a regular Raspberry Pi is connected."
- title: spark4pi-relay-actuator-2.3 -> spark4pi-digital-io-1.0

Commit message: Release spark4pi-digital-io-2.5
Parts:
- added C201, C202, C301, C302, C401, C402, C501, C502, C601, C602: 100nF, Capacitor_SMD:C_0402_1005Metric, symbol Device:C_Small
- added D201, D202, D301, D302, D401, D402, D501, D502, D601, D602: LED, LED_SMD:LED_0603_1608Metric, symbol Device:LED
- added D203, D303, D403, D503, D603: D_TVS, Resistor_SMD:R_0402_1005Metric, symbol Device:D_TVS
- added Q201, Q202, Q301, Q302, Q401, Q402, Q501, Q502, Q601, Q602: Q_NPN_BEC_BRT, Package_TO_SOT_SMD:SOT-323_SC-70, symbol Device:Q_NPN_BEC_BRT
- added R201, R202, R301, R302, R401, R402, R501, R502, R601, R602: 1K, Resistor_SMD:R_0402_1005Metric, symbol Device:R
- added R203, R303, R403, R503, R603: 51, Resistor_SMD:R_0805_2012Metric, symbol Device:R
- added R204, R304, R404, R504, R604: 10K, Resistor_SMD:R_0402_1005Metric, symbol Device:R
- added U201, U202, U301, U302, U401, U402, U501, U502, U601, U602: 74LVC1G125, Package_SO:TSOP-5_1.65x3.05mm_P0.95mm, symbol ice4pi:74LVC1G125
- added U203, U303, U403, U503, U603: SN74LVC1G14DBV, Package_TO_SOT_SMD:SOT-23-5, symbol 74xGxx:SN74LVC1G14DBV
- C101, C102: value 10uF -> 100nF
Connections:
- net +3V3: now also C201.1, C202.1, C301.1, C302.1, C401.1, C402.1, C501.1, C502.1, C601.1, C602.1, R201.1, R202.1, R204.1, R301.1, R302.1, R304.1, R401.1, R402.1, R404.1, R501.1, R502.1, R504.1, R601.1, R602.1, R604.1, U201.5 (VCC), U202.5 (VCC), U203.5 (VCC), U301.5 (VCC), U302.5 (VCC), U303.5 (VCC), U401.5 (VCC), U402.5 (VCC), U403.5 (VCC), U501.5 (VCC), U502.5 (VCC), U503.5 (VCC), U601.5 (VCC), U602.5 (VCC), U603.5 (VCC)
- net GND: now also C201.2, C202.2, C301.2, C302.2, C401.2, C402.2, C501.2, C502.2, C601.2, C602.2, D203.2 (A2), D303.2 (A2), D403.2 (A2), D503.2 (A2), D603.2 (A2), Q201.2 (E), Q202.2 (E), Q301.2 (E), Q302.2 (E), Q401.2 (E), Q402.2 (E), Q501.2 (E), Q502.2 (E), Q601.2 (E), Q602.2 (E), U201.3 (GND), U202.3 (GND), U203.3 (GND), U301.3 (GND), U302.3 (GND), U303.3 (GND), U401.3 (GND), U402.3 (GND), U403.3 (GND), U501.3 (GND), U502.3 (GND), U503.3 (GND), U601.3 (GND), U602.3 (GND), U603.3 (GND)
- net PORT2: now also Q201.1 (B), U201.2 (D), U202.4 (O)
- net PORT3: now also Q301.1 (B), U301.2 (D), U302.4 (O)
- net PORT4: now also Q401.1 (B), U401.2 (D), U402.4 (O)
- net PORT5: now also Q501.1 (B), U501.2 (D), U502.4 (O)
- net PORT6: now also Q601.1 (B), U601.2 (D), U602.4 (O)
- net PORT2_TX_ENABLE: now reaches P5.29 (GCLK1/GPIO5)
- net PORT2_TX_ENABLE: now also Q202.1 (B), R204.2, U202.1 (EN), U203.2
- net PORT3_TX_ENABLE: now reaches P5.31 (GCLK2/GPIO6)
- net PORT3_TX_ENABLE: now also Q302.1 (B), R304.2, U302.1 (EN), U303.2
- net PORT4_TX_ENABLE: now reaches P5.32 (PWM0/GPIO12)
- net PORT4_TX_ENABLE: now also Q402.1 (B), R404.2, U402.1 (EN), U403.2
- net PORT5_TX_ENABLE: now reaches P5.33 (PWM1/GPIO13)
- net PORT5_TX_ENABLE: now also Q502.1 (B), R504.2, U502.1 (EN), U503.2
- net PORT6_TX_ENABLE: now reaches P5.35 (GPIO19/MISO1)
- net PORT6_TX_ENABLE: now also Q602.1 (B), R604.2, U602.1 (EN), U603.2
- net at J501.1 (Pin_1): now also D503.1 (A1), R503.1
- net at J401.1 (Pin_1): now also D403.1 (A1), R403.1
- net at J601.1 (Pin_1): now also D603.1 (A1), R603.1
- net at J201.1 (Pin_1): now also D203.1 (A1), R203.1
- net at J301.1 (Pin_1): now also D303.1 (A1), R303.1
- new net: U601.1 (EN), U603.4
- new net: R603.2, U601.4 (O), U602.2 (D)
- new net: D401.1 (K), Q401.3 (C)
- new net: R503.2, U501.4 (O), U502.2 (D)
- new net: D501.2 (A), R501.2
- new net: D601.2 (A), R601.2
- new net: D201.1 (K), Q201.3 (C)
- new net: D201.2 (A), R201.2
- new net: U301.1 (EN), U303.4
- new net: R303.2, U301.4 (O), U302.2 (D)
- new net: U501.1 (EN), U503.4
- new net: U201.1 (EN), U203.4
- new net: R203.2, U201.4 (O), U202.2 (D)
- new net: D502.2 (A), R502.2
- new net: D601.1 (K), Q601.3 (C)
- new net: D202.1 (K), Q202.3 (C)
- new net: D401.2 (A), R401.2
- new net: D402.1 (K), Q402.3 (C)
- new net: D402.2 (A), R402.2
- new net: D602.1 (K), Q602.3 (C)
- new net: D602.2 (A), R602.2
- new net: U401.1 (EN), U403.4
- new net: D202.2 (A), R202.2
- new net: D302.1 (K), Q302.3 (C)
- new net: D302.2 (A), R302.2
- new net: R403.2, U401.4 (O), U402.2 (D)
- new net: D501.1 (K), Q501.3 (C)
- new net: D502.1 (K), Q502.3 (C)
- new net: D301.2 (A), R301.2
- new net: D301.1 (K), Q301.3 (C)
Other:
- title: spark4pi-digital-io-1.0 -> spark4pi-digital-io-2.5
- moved on the sheet: J301

Commit message: Release spark4pi-digital-io-2.6
Other:
- title: spark4pi-digital-io-2.5 -> spark4pi-digital-io-2.6
Changed lines of the file:
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@@
   (paper "A2")
   (title_block
-    (title "spark4pi-digital-io-2.5")
+    (title "spark4pi-digital-io-2.6")
     (company "Lightside Instruments AS")
   )

Commit message: Release spark4pi-digital-io-2.7
Other:
- title: spark4pi-digital-io-2.6 -> spark4pi-digital-io-2.7
Changed lines of the file:
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@@
   (paper "A2")
   (title_block
-    (title "spark4pi-digital-io-2.6")
+    (title "spark4pi-digital-io-2.7")
     (company "Lightside Instruments AS")
   )

Commit message: Release spark4pi-digital-io-2.8
Parts:
- added J3: Conn_01x03, Connector_PinHeader_2.54mm:PinHeader_1x03_P2.54mm_Vertical, symbol Connector_Generic:Conn_01x03
- D1: value LED -> LED_WHITE
- D101, D201, D301, D401, D501, D601: value LED -> LED_GREEN
- D102, D202, D302, D402, D502, D602: value LED -> LED_BLUE
- J2: value Conn_02x03 -> Conn_01x02
Connections:
- net +3V3: now also J3.3 (Pin_3); no longer C101.1, C201.1, C301.1, C401.1, C501.1, C601.1, U101.5 (VCC), U201.5 (VCC), U301.5 (VCC), U401.5 (VCC), U501.5 (VCC), U601.5 (VCC)
- net +5V: now also J3.1 (Pin_1)
- new net Vdrive: C101.1, C201.1, C301.1, C401.1, C501.1, C601.1, J3.2 (Pin_2), U101.5 (VCC), U201.5 (VCC), U301.5 (VCC), U401.5 (VCC), U501.5 (VCC), U601.5 (VCC)
Other:
- note added: "Jumper J2: Leave open (default) if a regular Raspberry Pi is connected. When closed the 2x20 Raspberry Pi 3.3V rail is powered from the LDO regulator on the extension board - 3V3 800 mA."
- note added: "Jumper J3: (1-2) +5V driver (default). 2.5V output when terminated with 50 ohm (2-3) +3.3V driver. 1.65V output when terminated with 50 ohm"
- note removed: "Jumper: Default open. Power the 2x20 Raspberry Pi 3.3V rail from the LDO regulator on the extension board - 3V3 800 mA. Leave open if a regular Raspberry Pi is connected."
- title: spark4pi-digital-io-2.7 -> spark4pi-digital-io-2.8

Commit message: Release spark4pi-digital-io-2.9
Other:
- title: spark4pi-digital-io-2.8 -> spark4pi-digital-io-2.9
Changed lines of the file:
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@@
   (paper "A2")
   (title_block
-    (title "spark4pi-digital-io-2.8")
+    (title "spark4pi-digital-io-2.9")
     (company "Lightside Instruments AS")
   )
