File: board/spark.kicad_sch (KiCad schematic)
At the start: 100 parts, among them J1 USB_C_Receptacle_USB2.0, J101 Conn_01x01_Shielded, J2 Conn_01x02, J201 Conn_01x01_Shielded, J3 Conn_01x03, J301 Conn_01x01_Shielded, J401 Conn_01x01_Shielded, J501 Conn_01x01_Shielded, J601 Conn_01x01_Shielded, P5 Raspberry_Pi_2_3, Q101 Q_NPN_BEC_BRT, Q102 Q_NPN_BEC_BRT, Q201 Q_NPN_BEC_BRT, Q202 Q_NPN_BEC_BRT, Q301 Q_NPN_BEC_BRT, Q302 Q_NPN_BEC_BRT, Q401 Q_NPN_BEC_BRT, Q402 Q_NPN_BEC_BRT, Q501 Q_NPN_BEC_BRT, Q502 Q_NPN_BEC_BRT, Q601 Q_NPN_BEC_BRT, Q602 Q_NPN_BEC_BRT, U1 LD1117S33TR_SOT223, U101 74LVC1G125, U102 74LVC1G125, U103 SN74LVC1G14DBV, U201 74LVC1G125, U202 74LVC1G125, U203 SN74LVC1G14DBV, U301 74LVC1G125, U302 74LVC1G125, U303 SN74LVC1G14DBV, U401 74LVC1G125, U402 74LVC1G125, U403 SN74LVC1G14DBV, U501 74LVC1G125, U502 74LVC1G125, U503 SN74LVC1G14DBV, U601 74LVC1G125, U602 74LVC1G125, U603 SN74LVC1G14DBV

Commit message: Release spark4pi-digital-io-2.10
Parts:
- removed U102, U202, U302, U402, U502, U602: 74LVC1G125, Package_SO:TSOP-5_1.65x3.05mm_P0.95mm, symbol ice4pi:74LVC1G125
- added C104, C204, C304, C404, C504, C604: 100nF, Capacitor_SMD:C_0402_1005Metric, symbol Device:C_Small
- added C3, C4: 10uF, Capacitor_SMD:C_0402_1005Metric, symbol Device:C_Small
- added J4: Conn_01x03, Connector_PinHeader_2.54mm:PinHeader_1x03_P2.54mm_Vertical, symbol Connector_Generic:Conn_01x03
- added R3: 220, Resistor_SMD:R_0402_1005Metric, symbol Device:R
- added R4: 68, Resistor_SMD:R_0402_1005Metric, symbol Device:R
- added R5: 5.1K, Resistor_SMD:R_0402_1005Metric, symbol Device:R
- added U102, U202, U302, U402, U502, U602: TXU0101DCK, Package_TO_SOT_SMD:SOT-363_SC-70-6, symbol spark:TXU0101DCK
- added U2: LM317_SOT-223, Package_TO_SOT_SMD:SOT-223-3_TabPin2, symbol Regulator_Linear:LM317_SOT-223
Connections:
- net +3V3: now also J4.3 (Pin_3), U102.6 (VCCB), U202.6 (VCCB), U302.6 (VCCB), U402.6 (VCCB), U502.6 (VCCB), U602.6 (VCCB)
- net +5V: now also C3.1, U2.3 (VI)
- net GND: now also C104.2, C204.2, C3.2, C304.2, C4.2, C404.2, C504.2, C604.2, R4.2, R5.2, U102.2 (GND), U202.2 (GND), U302.2 (GND), U402.2 (GND), U502.2 (GND), U602.2 (GND)
- net PORT1: now also U102.4 (BY)
- net PORT2: now also U202.4 (BY)
- net PORT3: now also U302.4 (BY)
- net PORT4: now also U402.4 (BY)
- net PORT5: now also U502.4 (BY)
- net PORT6: now also U602.4 (BY)
- net at U601.1 (EN), U603.4: now also U602.5 (OE)
- net at R603.2, U601.4 (O): now also U602.3 (A)
- net at R503.2, U501.4 (O): now also U502.3 (A)
- net at U301.1 (EN), U303.4: now also U302.5 (OE)
- net at R303.2, U301.4 (O): now also U302.3 (A)
- net at U501.1 (EN), U503.4: now also U502.5 (OE)
- net at U101.1 (EN), U103.4: now also U102.5 (OE)
- net at R103.2, U101.4 (O): now also U102.3 (A)
- net at U201.1 (EN), U203.4: now also U202.5 (OE)
- net at R203.2, U201.4 (O): now also U202.3 (A)
- net at J1.A5 (CC1), R2.1: no longer J1.B5 (CC2)
- net at U401.1 (EN), U403.4: now also U402.5 (OE)
- net at R403.2, U401.4 (O): now also U402.3 (A)
- new net: R3.2, R4.1, U2.1 (ADJ)
- new net: J1.B5 (CC2), R5.1
- new net +1V65: C4.1, J4.1 (Pin_1), R3.1, U2.2 (VO)
- new net Vrx: C104.1, C204.1, C304.1, C404.1, C504.1, C604.1, J4.2 (Pin_2), U102.1 (VCCA), U202.1 (VCCA), U302.1 (VCCA), U402.1 (VCCA), U502.1 (VCCA), U602.1 (VCCA)
Other:
- note added: "Jumper J3: (1-2) +5V driver (default). 2.5V output when terminated with 50 ohm. (2-3) +3.3V driver. 1.65V output when terminated with 50 ohm."
- note added: "Jumper J4: (1-2) +1.65V receiver. (2-3) +3.3V receiver (default)."
- note removed: "Jumper J3: (1-2) +5V driver (default). 2.5V output when terminated with 50 ohm (2-3) +3.3V driver. 1.65V output when terminated with 50 ohm"
- title: spark4pi-digital-io-2.9 -> spark4pi-digital-io-2.10
- moved on the sheet: R2
