File: board/spark_w_tstamp.kicad_pcb (KiCad board)
At the start: 4 copper layers, 198.5 x 85 mm, 44 parts, among them J10 Barrel_Jack, J101 Conn_01x01, J102 Conn_01x01, J103 Conn_01x01, J201 Conn_01x01, J202 Conn_01x01, J203 Conn_01x01, J3 Conn_02x06_Odd_Even, J301 Conn_01x01, J302 Conn_01x01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

Commit message: Release spark4pi-relay-actuator-2.0
Parts:
- removed the ? at (210.5, 76.0)
- removed the ? at (210.5, 45.0)
- removed the ? at (110.0, 76.0)
- removed the ? at (159.0, 76.0)
- removed the ? at (210.5, 107.5)
- removed the J102 at (98.5, 110.0)
- removed the R201 at (116.0, 87.2)
- removed REF**: Hole_2.5MM, spark:Hole_2.5MM
- added 1: Fiducial_1mm_Mask3mm, Fiducial:Fiducial_1mm_Mask3mm, F.Cu at (25.0, 44.5)
- added 2: Fiducial_1mm_Mask3mm, Fiducial:Fiducial_1mm_Mask3mm, F.Cu at (205.5, 122.5)
- added ?: , spark:mount_hole, F.Cu at (158.5, 77.5)
- added ?: , spark:mount_hole, F.Cu at (210.5, 102.5)
- added ?: , spark:mount_hole, F.Cu at (210.5, 122.5)
- added ?: , spark:mount_hole, F.Cu at (19.5, 122.5)
- added ?: , spark:mount_hole, F.Cu at (110.5, 77.5)
- added ?: , spark:mount_hole, F.Cu at (210.5, 44.5)
- added D202: LED, Diode_SMD:D_0603_1608Metric, F.Cu at (134.7, 125.0)
- added J103: Conn_01x01, spark:banana-plug-horizontal-black, F.Cu at (86.5, 57.0)
- R201: renamed from D202; value LED -> 10K; footprint Diode_SMD:D_0603_1608Metric -> Resistor_SMD:R_0402_1005Metric
- moved J102 54.3 mm to (98.5, 110.0), turned to 90 degrees
- moved R201 42.2 mm to (116.0, 87.2), turned to 0 degrees
- turned ? to 0 degrees
- renumbered J103 to J102
Connections:
- J102 pad 1: IN1 -> Net-(J102-Pad1)
- R201 pad 1: Net-(D202-Pad1) -> Net-(Q201-Pad1)
- R201 pad 2: SYS_DCIN -> GND
Other:
- board size 198.5 x 85 mm -> 198 x 85 mm
- board text added: "J103"
- board text added: "J203"
- board text added: "J303"
- board text added: "SPARK4PI-RELAY-ACTUATOR-2.0"
- board text removed: "SPARK4PI-RELAY-ACTUATOR-1.4"

Commit message: Release spark4pi-relay-actuator-2.1
Parts:
- removed the J201 at (122.5, 110.0)
- removed the R202 at (114.5, 87.7)
- added ?: , spark:mount_hole, F.Cu at (19.5, 102.5)
- added J302: Conn_01x01, spark:banana-plug-horizontal-black, F.Cu at (194.5, 110.0)
- J201: renamed from ?; value (none) -> Conn_01x01; footprint spark:mount_hole -> spark:banana-plug-horizontal-black
- R202: renamed from J302; value Conn_01x01 -> 1K; footprint spark:banana-plug-horizontal-black -> Resistor_SMD:R_0402_1005Metric
- moved J201 103.3 mm to (122.5, 110.0)
- moved R202 83.0 mm to (114.5, 87.7)
Connections:
- R202 pad 1: Net-(J302-Pad1) -> PORT2
Other:
- board text added: "SPARK4PI-RELAY-ACTUATOR-2.1"
- board text removed: "SPARK4PI-RELAY-ACTUATOR-2.0"
